Commit message: fix dumbell urdf

File: models/urdf/gen3_dumbbell.urdf (robot description, URDF)
Before this commit: robot GEN3_URDF_V12, 11 links, 10 joints
Links:
- removed link Base_Link
- removed link Bracelet_Link
- removed link EndEffector_Link
- removed link ForeArm_Link
- removed link HalfArm1_Link
- removed link HalfArm2_Link
- removed link Shoulder_Link
- removed link SphericalWrist1_Link
- removed link SphericalWrist2_Link
- added link base_link, mass 1.697; collision mesh filename=package://kortex_description/arms/gen3/7dof/meshes/base_lin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; visual mesh filename=package://kortex_description/arms/gen3/7dof/meshes/base_lin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
- added link bracelet_link, mass 0.5; collision mesh filename=package://kortex_description/arms/gen3/7dof/meshes/bracelet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; visual mesh filename=package://kortex_description/arms/gen3/7dof/meshes/bracelet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
- added link end_effector_link
- added link forearm_link, mass 0.9302; collision mesh filename=package://kortex_description/arms/gen3/7dof/meshes/forearm_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; visual mesh filename=package://kortex_description/arms/gen3/7dof/meshes/forearm_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
- added link gripper_left_coupler, mass 0.0273093985570947; collision mesh filename=package://Robotiq_2F85/meshes/left_coupler.STL; visual mesh filename=package://Robotiq_2F85/meshes/left_coupler.STL
- added link gripper_left_driver, mass 0.0184906489414316; collision mesh filename=package://Robotiq_2F85/meshes/left_driver.STL; visual mesh filename=package://Robotiq_2F85/meshes/left_driver.STL
- added link gripper_left_follower, mass 0.0195548943464751; collision mesh filename=package://Robotiq_2F85/meshes/left_follower.STL; visual mesh filename=package://Robotiq_2F85/meshes/left_follower.STL
- added link gripper_left_pad, mass 0.0112846745192961; collision mesh filename=package://Robotiq_2F85/meshes/left_pad.STL; visual mesh filename=package://Robotiq_2F85/meshes/left_pad.STL
- added link gripper_left_spring_link, mass 0.0299513316731757; collision mesh filename=package://Robotiq_2F85/meshes/left_spring_link.STL; visual mesh filename=package://Robotiq_2F85/meshes/left_spring_link.STL
- added link gripper_right_coupler, mass 0.0273093985570947; collision mesh filename=package://Robotiq_2F85/meshes/right_coupler.STL; visual mesh filename=package://Robotiq_2F85/meshes/right_coupler.STL
- added link gripper_right_driver, mass 0.0184906489409923; collision mesh filename=package://Robotiq_2F85/meshes/right_driver.STL; visual mesh filename=package://Robotiq_2F85/meshes/right_driver.STL
- added link gripper_right_follower, mass 0.0195548943464751; collision mesh filename=package://Robotiq_2F85/meshes/right_follower.STL; visual mesh filename=package://Robotiq_2F85/meshes/right_follower.STL
- added link gripper_right_pad, mass 0.0112846745192962; collision mesh filename=package://Robotiq_2F85/meshes/right_pad.STL; visual mesh filename=package://Robotiq_2F85/meshes/right_pad.STL
- added link gripper_right_spring_link, mass 0.029951; collision mesh filename=package://Robotiq_2F85/meshes/right_spring_link.STL; visual mesh filename=package://Robotiq_2F85/meshes/right_spring_link.STL
- added link half_arm_1_link, mass 1.1636; collision mesh filename=package://kortex_description/arms/gen3/7dof/meshes/half_arm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; visual mesh filename=package://kortex_description/arms/gen3/7dof/meshes/half_arm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
- added link half_arm_2_link, mass 1.1636; collision mesh filename=package://kortex_description/arms/gen3/7dof/meshes/half_arm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; visual mesh filename=package://kortex_description/arms/gen3/7dof/meshes/half_arm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
- added link shoulder_link, mass 1.3773; collision mesh filename=package://kortex_description/arms/gen3/7dof/meshes/shoulder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; visual mesh filename=package://kortex_description/arms/gen3/7dof/meshes/shoulder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
- added link spherical_wrist_1_link, mass 0.6781; collision mesh filename=package://kortex_description/arms/gen3/7dof/meshes/spherica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; visual mesh filename=package://kortex_description/arms/gen3/7dof/meshes/spherica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
- added link spherical_wrist_2_link, mass 0.6781; collision mesh filename=package://kortex_description/arms/gen3/7dof/meshes/spherica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; visual mesh filename=package://kortex_description/arms/gen3/7dof/meshes/spherica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
- link gripper_base: mass None -> 0.60831; geometry collision mesh filename=package://Robotiq_2F85/meshes/base.STL; visual mesh filename=package://Robotiq_2F85/meshes/base.STL
- link gripper_dumbbell_approx: mass 1.36078 -> 0.9072
Joints:
- removed joint Actuator1
- removed joint Actuator2
- removed joint Actuator3
- removed joint Actuator4
- removed joint Actuator5
- removed joint Actuator6
- removed joint Actuator7
- removed joint EndEffector
- added joint end_effector: type fixed, parent bracelet_link, child end_effector_link, origin xyz=0 0 -0.0615250000000001 rpy=3.14159265358979 1.09937075168372E-32 0, axis 0 0 0
- added joint gripper_left_coupler_joint: type fixed, parent gripper_left_driver, child gripper_left_coupler, origin xyz=0.031486 -0.0040855 0 rpy=3.1416 0 -3.1416, axis 0 0 1, limit lower=0.13 upper=0.79 effort=0 velocity=0
- added joint gripper_left_driver_joint: type fixed, parent gripper_base, child gripper_left_driver, origin xyz=-0.030601 -0.054792 0 rpy=0 0 -3.1245, axis 0 0 1, limit lower=-3.1416 upper=3.1416 effort=150 velocity=0
- added joint gripper_left_follower_joint: type fixed, parent gripper_left_coupler, child gripper_left_follower, origin xyz=-0.0061148 0.047125 0 rpy=0 0 0.017192, axis 0 0 1, limit lower=-3.1416 upper=3.1416 effort=0 velocity=0
- added joint gripper_left_pad_joint: type fixed, parent gripper_left_follower, child gripper_left_pad, origin xyz=0.018903 0.032265 0 rpy=0 0 -1.5708, axis 0 0 0
- added joint gripper_left_spring_link_joint: type fixed, parent gripper_base, child gripper_left_spring_link, origin xyz=-0.0127 -0.061307 0 rpy=3.1416 0 -0.70092, axis 0 0 1, limit lower=-0.7854 upper=0 effort=0 velocity=0
- added joint gripper_right_coupler_joint: type fixed, parent gripper_right_driver, child gripper_right_coupler, origin xyz=0.031486 -0.0040855 0 rpy=0 0 -0.25804, axis 0 0 -1, limit lower=0.13 upper=0.79 effort=0 velocity=0
- added joint gripper_right_driver_joint: type fixed, parent gripper_base, child gripper_right_driver, origin xyz=0.030601 -0.054792 0 rpy=3.1416 0 -0.019735, axis 0 0 1, limit lower=-3.1416 upper=3.1416 effort=150 velocity=0
- added joint gripper_right_follower_joint: type fixed, parent gripper_right_coupler, child gripper_right_follower, origin xyz=-0.0061148 0.047125 0 rpy=3.1416 0 -2.9033, axis 0 0 1, limit lower=-3.1416 upper=3.1416 effort=0 velocity=0
- added joint gripper_right_pad_joint: type fixed, parent gripper_right_follower, child gripper_right_pad, origin xyz=0.024903 0.032264 0 rpy=3.1416 0 -1.5708, axis 0 0 0
- added joint gripper_right_spring_link_joint: type fixed, parent gripper_base, child gripper_right_spring_link, origin xyz=0.0127 -0.061307 0 rpy=3.1416 0 0.6983, axis 0 0 1, limit lower=0 upper=0.7854 effort=0 velocity=0
- added joint joint_1: type revolute, parent base_link, child shoulder_link, origin xyz=0 0 0.15643 rpy=3.1416 2.7629E-18 -4.9305E-36, axis 0 0 1, limit lower=-1000.0 upper=1000.0 effort=39 velocity=1.3963
- added joint joint_2: type revolute, parent shoulder_link, child half_arm_1_link, origin xyz=0 0.005375 -0.12838 rpy=1.5708 2.1343E-17 -1.1102E-16, axis 0 0 1, limit lower=-2.41 upper=2.41 effort=39 velocity=1.3963
- added joint joint_3: type revolute, parent half_arm_1_link, child half_arm_2_link, origin xyz=0 -0.21038 -0.006375 rpy=-1.5708 1.2326E-32 -2.9122E-16, axis 0 0 1, limit lower=-1000.0 upper=1000.0 effort=39 velocity=1.3963
- added joint joint_4: type revolute, parent half_arm_2_link, child forearm_link, origin xyz=0 0.006375 -0.21038 rpy=1.5708 -6.6954E-17 -1.6653E-16, axis 0 0 1, limit lower=-2.66 upper=2.66 effort=39 velocity=1.3963
- added joint joint_5: type revolute, parent forearm_link, child spherical_wrist_1_link, origin xyz=0 -0.20843 -0.006375 rpy=-1.5708 2.2204E-16 -6.373E-17, axis 0 0 1, limit lower=-1000.0 upper=1000.0 effort=9 velocity=1.2218
- added joint joint_6: type revolute, parent spherical_wrist_1_link, child spherical_wrist_2_link, origin xyz=0 0.00017505 -0.10593 rpy=1.5708 9.2076E-28 -8.2157E-15, axis 0 0 1, limit lower=-2.23 upper=2.23 effort=9 velocity=1.2218
- added joint joint_7: type revolute, parent spherical_wrist_2_link, child bracelet_link, origin xyz=0 -0.10593 -0.00017505 rpy=-1.5708 -5.5511E-17 9.6396E-17, axis 0 0 1, limit lower=-1000.0 upper=1000.0 effort=9 velocity=1.2218
- joint gripper_base_joint: origin xyz=0.0 0.0 -0.0615250000000001 rpy=1.5707 0.0 0.0 -> xyz=0.0 0.0 0.0 rpy=0.0 0.0 1.57; parent Bracelet_Link -> end_effector_link
- joint gripper_dumbbell_joint: origin xyz=0.0 -0.10155 0 rpy=0.0 0.0 0.0 -> xyz=-0.005 -0.16 0.025 rpy=0 1.5707 0
