Commit message: update urdf with dumbbells

File: models/urdf/gen3_2f85_dumbbell_4lb.urdf (robot description, URDF)
Before this commit: robot gen3_2f85_dumbbell_4lb, 22 links, 21 joints
Links:
- link object_link: geometry collision mesh filename=meshes/dumbbell_4lb.STL scale=0.001 0.001 0.001; visual mesh filename=meshes/dumbbell_4lb.STL scale=0.001 0.001 0.001

File: models/urdf/gen3_2f85_dumbbell_5lb.urdf (robot description, URDF)
Before this commit: robot gen3_2f85_dumbbell_5lb, 22 links, 21 joints
Links:
- link object_link: geometry collision mesh filename=meshes/dumbbell_5lb.STL scale=0.001 0.001 0.001; visual mesh filename=meshes/dumbbell_5lb.STL scale=0.001 0.001 0.001

File: models/urdf/gen3_2f85_dumbbell_7lb.urdf (robot description, URDF)
Before this commit: robot gen3_2f85_dumbbell_6lb, 22 links, 21 joints
Links:
- link object_link: geometry collision mesh filename=meshes/dumbbell_7lb.STL scale=0.001 0.001 0.001; visual mesh filename=meshes/dumbbell_7lb.STL scale=0.001 0.001 0.001

File: models/urdf/gen3_2f85_dumbbell_8lb.urdf (robot description, URDF)
Before this commit: robot gen3_2f85_dumbbell_6lb, 22 links, 21 joints
Links:
- link object_link: mass 2.72155422 -> 3.17514659; geometry collision mesh filename=meshes/dumbbell_8lb.STL scale=0.001 0.001 0.001; visual mesh filename=meshes/dumbbell_8lb.STL scale=0.001 0.001 0.001
