Commit message: update urdf and install description

File: models/urdf/kinova_with_suction.urdf (robot description, URDF)
Before this commit: robot kinova-gen3-with-suction, 8 links, 7 joints
Links:
- link base_link: geometry collision mesh filename=meshes/base_link.stl; visual mesh filename=meshes/base_link.stl
- link bracelet_link: geometry collision mesh filename=meshes/bracelet_with_suction_gripper.stl; visual mesh filename=meshes/bracelet_with_suction_gripper.stl
- link forearm_link: geometry collision mesh filename=meshes/forearm_link.stl; visual mesh filename=meshes/forearm_link.stl
- link half_arm_1_link: geometry collision mesh filename=meshes/half_arm_1_link.stl; visual mesh filename=meshes/half_arm_1_link.stl
- link half_arm_2_link: geometry collision mesh filename=meshes/half_arm_2_link.stl; visual mesh filename=meshes/half_arm_2_link.stl
- link shoulder_link: geometry collision mesh filename=meshes/shoulder_link.stl; visual mesh filename=meshes/shoulder_link.stl
- link spherical_wrist_1_link: geometry collision mesh filename=meshes/spherical_wrist_1_link.stl; visual mesh filename=meshes/spherical_wrist_1_link.stl
- link spherical_wrist_2_link: geometry collision mesh filename=meshes/spherical_wrist_2_link.stl; visual mesh filename=meshes/spherical_wrist_2_link.stl
